File: DesignBlockskicad_blocks.kicad_blocks/CH572D.kicad_block/CH572D.kicad_sch (KiCad schematic)
At the start: 8 parts, among them Y1 32mhz

Commit message: a whole bunch of designs
Connections:
- net +3.3V is gone; now on net PWR_3V3: S1.1, S1.2
- net GND is gone; now on net PWR_GND: C5.2, C6.2, C7.2
Other:
- moved on the sheet: E1
